File: board/board.kicad_pcb (KiCad board)
At the start: 2 copper layers, 43.7 x 39.1 mm, 22 parts, among them J1 AVR-ISP-10, J2 Conn_02x18_Top_Bottom, Q1 BSS138, Q2 BSS138, Q3 BC847, U1 AP1117-33, U2 ESP-01v090, U3 ATmega328P-AU, Y1 10MHz

Commit message: Use 16MHz crystal on schematics
Parts:
- Y1: value 10MHz -> 16MHz
Changed lines of the file:
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@@
   (page A4)
   (layers
-    (0 F.Cu signal)
+    (0 F.Cu signal hide)
     (31 B.Cu signal)
     (32 B.Adhes user)
@@
       (effects (font (size 1 1) (thickness 0.15)))
     )
-    (fp_text value 10MHz (at 9.275 3.3125 90) (layer F.Fab)
-      (effects (font (size 1 1) (thickness 0.15)))
-    )
+    (fp_text value 16MHz (at 9.275 3.3125 90) (layer F.Fab)
+      (effects (font (size 1 1) (thickness 0.15)))
+    )
